File: projects/blizzard/s2mod/tower.kicad_sch (KiCad schematic)
At the start: 19 parts, among them U1 S2MOD_REV, U3 BALF-SPI2-01D3, Y1 24M

Commit message: Fix balun rotation in JLCPCB exports
Parts:
- U3: JLCPCB_CORRECTION (none) -> 0;0;-90
Changed lines of the file:
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@@
       (effects (font (size 1.27 1.27)) (justify bottom) hide)
+    )
+    (property "JLCPCB_CORRECTION" "0;0;-90" (at 193.04 62.23 0)
+      (effects (font (size 1.27 1.27)) hide)
     )
     (pin "A1")
