File: projects/blizzard/s2mod/tower.kicad_sch (KiCad schematic)
At the start: 19 parts, among them U1 S2MOD_REV, U3 BALF-SPI2-01D3, Y1 24M

Commit message: Update part number for inductors
Parts:
- L1: LCSC C1035 -> C84474
Changed lines of the file:
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@@
       (effects (font (size 1.27 1.27)) hide)
     )
-    (property "LCSC" "C1035" (at 158.75 88.9 0)
+    (property "LCSC" "C84474" (at 158.75 88.9 0)
       (effects (font (size 1.27 1.27)) hide)
     )

Commit message: Fix balun rotation in JLCPCB exports and change to LGA
Parts:
- removed H1, H2, H3, H4: Tabs, kikit:Tab, symbol Mechanical:MountingHole
- U3: JLCPCB_CORRECTION (none) -> 0;0;-90
Changed lines of the file:
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@@
-    )
-  )
-  (symbol (lib_id "Mechanical:MountingHole") (at 58.42 92.71 0) (unit 1)
-    (in_bom yes) (on_board yes) (dnp no) (fields_autoplaced)
-    (property "Reference" "H1" (at 60.96 91.44 0)
-      (effects (font (size 1.27 1.27)) (justify left))
-    )
-    (property "Value" "Tabs" (at 60.96 93.98 0)
-      (effects (font (size 1.27 1.27)) (justify left))
-    )
-    (property "Footprint" "kikit:Tab" (at 58.42 92.71 0)
-      (effects (font (size 1.27 1.27)) hide)
-    )
-    (property "Datasheet" "~" (at 58.42 92.71 0)
-      (effects (font (size 1.27 1.27)) hide)
-    )
-    (instances
-      (project "tower"
-        (path "/a1f46c5a-a489-4b1d-b2aa-fa6c12b9b1a3"
-          (reference "H1") (unit 1)
-        )
-      )
     )
   )
@@
         (path "/a1f46c5a-a489-4b1d-b2aa-fa6c12b9b1a3"
           (reference "#PWR011") (unit 1)
-        )
-      )
-    )
-  )
-  (symbol (lib_id "Mechanical:MountingHole") (at 58.42 102.87 0) (unit 1)
-    (in_bom yes) (on_board yes) (dnp no) (fields_autoplaced)
-    (property "Reference" "H3" (at 60.96 101.6 0)
-      (effects (font (size 1.27 1.27)) (justify left))
-    )
-    (property "Value" "Tabs" (at 60.96 104.14 0)
-      (effects (font (size 1.27 1.27)) (justify left))
-    )
-    (property "Footprint" "kikit:Tab" (at 58.42 102.87 0)
-      (effects (font (size 1.27 1.27)) hide)
-    )
-    (property "Datasheet" "~" (at 58.42 102.87 0)
-      (effects (font (size 1.27 1.27)) hide)
-    )
-    (instances
-      (project "tower"
-        (path "/a1f46c5a-a489-4b1d-b2aa-fa6c12b9b1a3"
-          (reference "H3") (unit 1)
         )
       )
@@
       (effects (font (size 1.27 1.27)) (justify bottom) hide)
     )
+    (property "JLCPCB_CORRECTION" "0;0;-90" (at 193.04 62.23 0)
+      (effects (font (size 1.27 1.27)) hide)
+    )
     (pin "A1")
     (pin "A2")
@@
         )
       )
-    )
-  )
-  (symbol (lib_id "Mechanical:MountingHole") (at 69.85 102.87 0) (unit 1)
-    (in_bom yes) (on_board yes) (dnp no) (fields_autoplaced)
-    (property "Reference" "H4" (at 72.39 101.6 0)
-      (effects (font (size 1.27 1.27)) (justify left))
-    )
-    (property "Value" "Tabs" (at 72.39 104.14 0)
-      (effects (font (size 1.27 1.27)) (justify left))
-    )
-    (property "Footprint" "kikit:Tab" (at 69.85 102.87 0)
-      (effects (font (size 1.27 1.27)) hide)
-    )
-    (property "Datasheet" "~" (at 69.85 102.87 0)
-      (effects (font (size 1.27 1.27)) hide)
-    )
-    (instances
-      (project "tower"
-        (path "/a1f46c5a-a489-4b1d-b2aa-fa6c12b9b1a3"
-          (reference "H4") (unit 1)
-        )
-      )
-    )
-  )
-  (symbol (lib_id "Mechanical:MountingHole") (at 69.85 92.71 0) (unit 1)
-    (in_bom yes) (on_board yes) (dnp no) (fields_autoplaced)
-    (property "Reference" "H2" (at 72.39 91.44 0)
-      (effects (font (size 1.27 1.27)) (justify left))
-    )
-    (property "Value" "Tabs" (at 72.39 93.98 0)
-      (effects (font (size 1.27 1.27)) (justify left))
-    )
-    (property "Footprint" "kikit:Tab" (at 69.85 92.71 0)
-      (effects (font (size 1.27 1.27)) hide)
-    )
-    (property "Datasheet" "~" (at 69.85 92.71 0)
-      (effects (font (size 1.27 1.27)) hide)
-    )
-    (instances
-      (project "tower"
-        (path "/a1f46c5a-a489-4b1d-b2aa-fa6c12b9b1a3"
-          (reference "H2") (unit 1)
-        )
-      )
